Commit message: .

File: peg_in_hole/urdf/Three/socket_wall_three.xacro (robot description, xacro)
@@ -16,5 +16,5 @@
 		<origin xyz="0 0 0" rpy="0 0 0"/>
 		<geometry>
-   			<mesh filename="package://objects/meshes/${socket_t}/${socket_t}.dae"/>
+   			<mesh filename="package://objects/meshes/${socket_t}/${socket_t}.dae" scale="0.9 1 1"/>
 		</geometry>
         </visual>

File: peg_in_hole/urdf/Two/socket_wall_two.xacro (robot description, xacro)
@@ -36,5 +36,5 @@
 	</xacro:if>
 	<xacro:if value="${use_socket_two}">
-		<origin xyz="${-0.0025} 0 0" rpy="0 0 ${-M_PI/2}"/>
+		<origin xyz="${-0.038} 0 0.0" rpy="0 0 ${-M_PI/2}"/>
 	</xacro:if>
 	<xacro:if value="${use_socket_three}">

File: peg_in_hole/urdf/Two/table_sw_two.xacro (robot description, xacro)
@@ -4,5 +4,4 @@
 <xacro:include filename="$(find peg_in_hole)/urdf/Two/socket_wall_two.xacro" />
 <joint name="link_table_wall" type="fixed">
-	<!-- " r-->
 	<origin xyz="0 ${-0.24 + 0.03} ${-0.2 - 0.04}" rpy="0 0 ${M_PI/2}"/>
 	<parent link="link_wall"/>
